File: Compressor.kicad_sch (KiCad schematic)
At the start: 32 parts, among them Q401 2N5457, U401 TL072

Commit message: Added schematic, assembly drawings, and assembly BoM exports
Parts:
- C401: Source (none) -> MOUSER: 810-FG18C0G1H101JNT0
- C402: Source (none) -> MOUSER: 810-FG14C0G1H333JNT6
- C403: Source (none) -> MOUSER: 810-FG28C0G1H152JNT6
- C404: Source (none) -> MOUSER: 810-FG14X7R1H224KNT0
- C405, C407, C410: Source (none) -> MOUSER: 667-EEA-FC1E100
- C406: Source (none) -> MOUSER: 594-K153K15X7RF53L2
- C408, C409: Source (none) -> MOUSER: 232-25PX100MEFC5X11
- D401, D402: Source (none) -> MOUSER: 606-4304H1
- D403: Part No. BAR43SFILM -> (none); PartNo. (none) -> BAR43SFILM; Source (none) -> MOUSER: 511-BAR43SFILM
- Q401: Source (none) -> https://stompboxparts.com/semiconductors/2n5457-jfet/
- R401, R415: Source (none) -> MOUSER: 603-MFR-25FBF52-200R
- R402, R403, R404, R410, R412: Source (none) -> MOUSER: 603-MFR-25FTF52-1M
- R405, R409: Source (none) -> MOUSER: 603-MFR-25FTF52-10K
- R406, R413: Source (none) -> MOUSER: 603-MFR-25FBF52-39K
- R407, R411: Source (none) -> MOUSER: 603-MFR-25FBF52-22R
- R408: Source (none) -> MOUSER: 603-MFR-25FBF52-5K1
- R414: Source (none) -> MOUSER: 603-MFR-25FBF52-47K
- RV401, RV402: Source (none) -> MOUSER: 306-B3BXHALFSNP
- U401: Source (none) -> MOUSER: 595-TL072CP
