File: Equalizer.kicad_sch (KiCad schematic)
At the start: 11 parts, among them U501 TL072

Commit message: Added schematic, assembly drawings, and assembly BoM exports
Parts:
- C501: PartNo. (none) -> FG14C0G1H333JNT06; Source (none) -> MOUSER: 810-FG14C0G1H333JNT6
- C502: Source (none) -> MOUSER: 810-FG18X7R1H473KNT6
- R501, R504: Source (none) -> MOUSER: 603-MFR-25FTF52-22K
- R503: Source (none) -> MOUSER: 603-MFR-25FBF52-220K
- R505: Source (none) -> MOUSER: 603-MFR-25FRF5215K
- R506: Source (none) -> MOUSER: 603-MFR-25FTF52-10K
- R507: Source (none) -> MOUSER: 603-MFR-25FBF52-1K
- RV501, RV502: Source (none) -> MOUSER: 306-B3BXHALFSNP
- U501: Source (none) -> MOUSER: 595-TL072CP
Changed lines of the file:
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@@
+			)
+		)
+		(property "Source" "MOUSER: 603-MFR-25FBF52-220K"
+			(at 82.55 44.45 0)
+			(effects
+				(font
+					(size 1.27 1.27)
+				)
+				(hide yes)
 			)
 		)
@@
 			)
 		)
+		(property "Source" "MOUSER: 595-TL072CP"
+			(at 90.17 82.55 0)
+			(effects
+				(font
+					(size 1.27 1.27)
+				)
+				(hide yes)
+			)
+		)
 		(pin "3"
 		)
@@
 			)
 		)
+		(property "Source" "MOUSER: 603-MFR-25FTF52-22K"
+			(at 77.47 35.56 0)
+			(effects
+				(font
+					(size 1.27 1.27)
+				)
+				(hide yes)
+			)
+		)
 		(pin "2"
 		)
@@
 			)
 		)
+		(property "PartNo." "FG14C0G1H333JNT06"
+			(at 71.12 54.61 0)
+			(effects
+				(font
+					(size 1.27 1.27)
+				)
+				(hide yes)
+			)
+		)
+		(property "Source" "MOUSER: 810-FG14C0G1H333JNT6 "
+			(at 71.12 54.61 0)
+			(effects
+				(font
+					(size 1.27 1.27)
+				)
+				(hide yes)
+			)
+		)
 		(pin "1"
 		)
@@
 			)
 		)
+		(property "Source" "MOUSER: 810-FG18X7R1H473KNT6 "
+			(at 77.47 63.5 0)
+			(effects
+				(font
+					(size 1.27 1.27)
+				)
+				(hide yes)
+			)
+		)
 		(pin "1"
 		)
@@
 			)
 		)
+		(property "Source" "MOUSER: 603-MFR-25FTF52-10K"
+			(at 114.3 95.25 0)
+			(effects
+				(font
+					(size 1.27 1.27)
+				)
+				(hide yes)
+			)
+		)
 		(pin "2"
 		)
@@
 			)
 		)
+		(property "Source" "MOUSER: 603-MFR-25FTF52-22K"
+			(at 100.33 35.56 0)
+			(effects
+				(font
+					(size 1.27 1.27)
+				)
+				(hide yes)
+			)
+		)
 		(pin "2"
 		)
@@
 			)
 		)
+		(property "Source" "MOUSER: 306-B3BXHALFSNP"
+			(at 54.61 26.67 0)
+			(effects
+				(font
+					(size 1.27 1.27)
+				)
+				(hide yes)
+			)
+		)
 		(pin "3"
 		)
@@
 			)
 		)
+		(property "Source" "MOUSER: 595-TL072CP"
+			(at 27.94 58.42 0)
+			(effects
+				(font
+					(size 1.27 1.27)
+				)
+				(hide yes)
+			)
+		)
 		(pin "3"
 		)
@@
 		)
 		(property "Sim.Type" ""
+			(at 107.95 64.77 0)
+			(effects
+				(font
+					(size 1.27 1.27)
+				)
+				(hide yes)
+			)
+		)
+		(property "Source" "MOUSER: 603-MFR-25FBF52-1K"
 			(at 107.95 64.77 0)
 			(effects
@@
 			)
 		)
+		(property "Source" "MOUSER: 595-TL072CP"
+			(at 100.33 52.07 0)
+			(effects
+				(font
+					(size 1.27 1.27)
+				)
+				(hide yes)
+			)
+		)
 		(pin "3"
 		)
@@
 			)
 		)
+		(property "Source" "MOUSER: 603-MFR-25FRF5215K"
+			(at 60.96 54.61 0)
+			(effects
+				(font
+					(size 1.27 1.27)
+				)
+				(hide yes)
+			)
+		)
 		(pin "2"
 		)
@@
 			(at 114.3 80.01 0)
 			(effects
+				(font
+					(size 1.27 1.27)
+				)
+				(hide yes)
+			)
+		)
+		(property "Source" "MOUSER: 306-B3BXHALFSNP"
+			(at 114.3 80.01 0)
+			(effects
