File: Fuzz.kicad_sch (KiCad schematic)
At the start: 11 parts, among them Q701 BC109, Q702 BC109

Commit message: Added schematic, assembly drawings, and assembly BoM exports
Parts:
- C701, C703: Source (none) -> MOUSER: 667-ECA-1HM2R2
- C702: Source (none) -> MOUSER: 810-FG28C0G1H103JNT6
- Q701, Q702: Source (none) -> MOUSER: 610-BC109C-TL
- R701: Source (none) -> MOUSER: 603-MFR-25FBF52-8K2
- R702: Source (none) -> MOUSER: 603-MFR-25FTF52-330R
- R703: Source (none) -> MOUSER: 603-MFR-25FBF52-33K
- R704: Source (none) -> MOUSER: 708-RNF14FTD100K
- RV701, RV702: Source (none) -> MOUSER: 306-B3BXHALFSNP
Changed lines of the file:
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@@
+			)
+		)
+		(property "Source" "MOUSER: 306-B3BXHALFSNP"
+			(at 105.41 87.63 0)
+			(effects
+				(font
+					(size 1.27 1.27)
+				)
+				(hide yes)
 			)
 		)
@@
 			)
 		)
+		(property "Source" "MOUSER: 603-MFR-25FBF52-8K2"
+			(at 97.79 40.64 0)
+			(effects
+				(font
+					(size 1.27 1.27)
+				)
+				(hide yes)
+			)
+		)
 		(pin "1"
 		)
@@
 			)
 		)
+		(property "Source" "MOUSER: 667-ECA-1HM2R2"
+			(at 59.69 64.77 0)
+			(effects
+				(font
+					(size 1.27 1.27)
+				)
+				(hide yes)
+			)
+		)
 		(pin "1"
 		)
@@
 			)
 		)
+		(property "Source" "MOUSER: 603-MFR-25FBF52-33K"
+			(at 78.74 40.64 0)
+			(effects
+				(font
+					(size 1.27 1.27)
+				)
+				(hide yes)
+			)
+		)
 		(pin "1"
 		)
@@
 			)
 		)
+		(property "Source" "MOUSER: 603-MFR-25FTF52-330R "
+			(at 90.17 31.75 0)
+			(effects
+				(font
+					(size 1.27 1.27)
+				)
+				(hide yes)
+			)
+		)
 		(pin "1"
 		)
@@
 			)
 		)
+		(property "Source" "MOUSER: 810-FG28C0G1H103JNT6"
+			(at 109.22 31.75 0)
+			(effects
+				(font
+					(size 1.27 1.27)
+				)
+				(hide yes)
+			)
+		)
 		(pin "1"
 		)
@@
 			)
 		)
+		(property "Source" "MOUSER: 610-BC109C-TL "
+			(at 76.2 64.77 0)
+			(effects
+				(font
+					(size 1.27 1.27)
+				)
+				(hide yes)
+			)
+		)
 		(pin "3"
 		)
@@
 			)
 		)
+		(property "Source" "MOUSER: 667-ECA-1HM2R2"
+			(at 115.57 80.01 0)
+			(effects
+				(font
+					(size 1.27 1.27)
+				)
+				(hide yes)
+			)
+		)
 		(pin "1"
 		)
@@
 			)
 		)
+		(property "Source" "MOUSER: 306-B3BXHALFSNP"
+			(at 123.19 41.91 0)
+			(effects
+				(font
+					(size 1.27 1.27)
+				)
+				(hide yes)
+			)
+		)
 		(pin "3"
 		)
@@
 			)
 		)
+		(property "Source" "MOUSER: 708-RNF14FTD100K"
+			(at 67.31 72.39 0)
+			(effects
+				(font
+					(size 1.27 1.27)
+				)
+				(hide yes)
+			)
+		)
 		(pin "1"
 		)
@@
 			(at 95.25 50.8 0)
 			(effects
+				(font
+					(size 1.27 1.27)
+				)
+				(hide yes)
+			)
+		)
+		(property "Source" "MOUSER: 610-BC109C-TL "
+			(at 95.25 50.8 0)
+			(effects
